File: Ergokyle-PCB.kicad_sch (KiCad schematic)
At the start: 162 parts, among them J1 Conn_01x12, J2 OLED, J3 Conn_01x12, J4 AudioJack4, J5 Conn_01x12, J6 Conn_01x12, J7 Conn_01x05, J8 AudioJack4, J9 Cirque_TRKPD, SW1 RotaryEncoder_Switch, SW2 SW_Push, SW3 RotaryEncoder_Switch, SW4 RotaryEncoder_Switch

Commit message: PCB file update
Parts:
- J1, J3, J5, J6: footprint (none) -> Connector_PinSocket_2.54mm:PinSocket_1x12_P2.54mm_Vertical
- J2, J9: footprint (none) -> Connector_PinSocket_2.54mm:PinSocket_1x04_P2.54mm_Vertical
- J4, J8: footprint (none) -> Connector_Audio:Jack_3.5mm_PJ320E_Horizontal
- J7: footprint (none) -> Connector_PinSocket_2.54mm:PinSocket_1x05_P2.54mm_Vertical
- MX1, MX10, MX11, MX12, MX13, MX14, MX15, MX16, MX17, MX18, MX19, MX2, MX20, MX21, MX22, MX23, MX24, MX25, MX26, MX27, MX28, MX29, MX3, MX30, MX31, MX32, MX33, MX34, MX35, MX36, MX37, MX39, MX4, MX41, MX42, MX43, MX44, MX45, MX46, MX48, MX49, MX5, MX50, MX51, MX52, MX53, MX54, MX55, MX56, MX57, MX58, MX59, MX6, MX60, MX61, MX62, MX63, MX64, MX65, MX66, MX68, MX69, MX7, MX71, MX72, MX73, MX74, MX75, MX76, MX8, MX9: footprint MX_Alps_Hybrid:MX-1U -> PCM_marbastlib-mx:SW_MX_HS_CPG151101S11_1u
- MX40, MX67: footprint MX_Alps_Hybrid:MX-1.25U -> PCM_marbastlib-mx:SW_MX_HS_CPG151101S11_1.25u
- SW1, SW3: footprint (none) -> random-keyboard-parts:RollerEncoder_Panasonic_EVQWGD001
- SW2: footprint (none) -> Kailh red micro switch silent:Kailh red micro switch silent
- SW4: footprint (none) -> random-keyboard-parts:RotaryEncoder_Alps_EC11E-Switch_Vertical_H20mm_MountingHoles
Connections:
- net at MX4.2 (ROW): now also D4.2 (A); no longer D4.1 (K)
- net at D40.1 (K): now also D33.1 (K), D34.1 (K), D35.1 (K), D36.1 (K), D37.1 (K), D38.1 (K), D39.1 (K), J3.11 (Pin_11); no longer MX40.2 (ROW)
- net at D68.1 (K): now also D67.1 (K), D69.1 (K), D70.1 (K), D71.1 (K), D72.1 (K), D74.1 (K), J5.11 (Pin_11); no longer MX68.2 (ROW)
- net at MX1.2 (ROW): now also D1.2 (A); no longer D1.1 (K)
- net at MX30.2 (ROW): now also D30.2 (A); no longer D30.1 (K)
- net at MX74.2 (ROW): now also D74.2 (A); no longer D74.1 (K)
- net at MX22.2 (ROW): now also D22.2 (A); no longer D22.1 (K)
- net at MX18.2 (ROW): now also D18.2 (A); no longer D18.1 (K)
- net at MX52.2 (ROW): now also D52.2 (A); no longer D52.1 (K)
- net at D21.1 (K): now also D17.1 (K), D18.1 (K), D19.1 (K), D20.1 (K), D22.1 (K), D23.1 (K), D24.1 (K), J3.9 (Pin_9); no longer MX21.2 (ROW)
- net at D12.1 (K): now also D10.1 (K), D11.1 (K), D13.1 (K), D14.1 (K), D15.1 (K), D16.1 (K), D9.1 (K), J3.8 (Pin_8); no longer MX12.2 (ROW)
- net at MX58.2 (ROW): now also D58.2 (A); no longer D58.1 (K)
- net at MX44.2 (ROW): now also D44.2 (A); no longer D44.1 (K)
- net at D51.1 (K): now also D48.1 (K), D49.1 (K), D50.1 (K), D52.1 (K), D53.1 (K), D54.1 (K), J5.6 (Pin_6); no longer MX51.2 (ROW)
- net at D25.1 (K): now also D26.1 (K), D27.1 (K), D28.1 (K), D29.1 (K), D30.1 (K), D31.1 (K), D32.1 (K), J3.10 (Pin_10); no longer MX25.2 (ROW)
- net at MX48.2 (ROW): now also D48.2 (A); no longer D48.1 (K)
- net at D46.1 (K): now also D41.1 (K), D42.1 (K), D43.1 (K), D44.1 (K), D45.1 (K), D47.1 (K), J5.5 (Pin_5); no longer MX46.2 (ROW)
- net at MX34.2 (ROW): now also D34.2 (A); no longer D34.1 (K)
- net at MX36.2 (ROW): now also D36.2 (A); no longer D36.1 (K)
- net at MX64.2 (ROW): now also D64.2 (A); no longer D64.1 (K)
- net at SW1.S2: now also D38.2 (A); no longer D38.1 (K)
- net at MX24.2 (ROW): now also D24.2 (A); no longer D24.1 (K)
- net at D60.1 (K): now also D55.1 (K), D56.1 (K), D57.1 (K), D58.1 (K), D59.1 (K), D75.1 (K), J5.9 (Pin_9); no longer MX60.2 (ROW)
- net at MX20.2 (ROW): now also D20.2 (A); no longer D20.1 (K)
- net at MX76.2 (ROW): now also D76.2 (A); no longer D76.1 (K)
- net at MX53.2 (ROW): now also D53.2 (A); no longer D53.1 (K)
- net at MX62.2 (ROW): now also D62.2 (A); no longer D62.1 (K)
- net at MX50.2 (ROW): now also D50.2 (A); no longer D50.1 (K)
- net at MX29.2 (ROW): now also D29.2 (A); no longer D29.1 (K)
- net at MX13.2 (ROW): now also D13.2 (A); no longer D13.1 (K)
- net at MX23.2 (ROW): now also D23.2 (A); no longer D23.1 (K)
- net at D5.1 (K): now also D1.1 (K), D2.1 (K), D3.1 (K), D4.1 (K), D6.1 (K), D7.1 (K), D8.1 (K), J3.7 (Pin_7); no longer MX5.2 (ROW)
- net at MX26.2 (ROW): now also D26.2 (A); no longer D26.1 (K)
- net at MX71.2 (ROW): now also D71.2 (A); no longer D71.1 (K)
- net at MX49.2 (ROW): now also D49.2 (A); no longer D49.1 (K)
- net at MX16.2 (ROW): now also D16.2 (A); no longer D16.1 (K)
- net at D63.1 (K): now also D61.1 (K), D62.1 (K), D64.1 (K), D65.1 (K), D66.1 (K), D73.1 (K), D76.1 (K), J5.10 (Pin_10); no longer MX63.2 (ROW)
- net at MX45.2 (ROW): now also D45.2 (A); no longer D45.1 (K)
- net at MX69.2 (ROW): now also D69.2 (A); no longer D69.1 (K)
- net at MX54.2 (ROW): now also D54.2 (A); no longer D54.1 (K)
- net at MX66.2 (ROW): now also D66.2 (A); no longer D66.1 (K)
- net at MX37.2 (ROW): now also D37.2 (A); no longer D37.1 (K)
- net at SW3.S2: now also D70.2 (A); no longer D70.1 (K)
- net at MX11.2 (ROW): now also D11.2 (A); no longer D11.1 (K)
- net at MX10.2 (ROW): now also D10.2 (A); no longer D10.1 (K)
- net at MX7.2 (ROW): now also D7.2 (A); no longer D7.1 (K)
- net at MX27.2 (ROW): now also D27.2 (A); no longer D27.1 (K)
- net at MX35.2 (ROW): now also D35.2 (A); no longer D35.1 (K)
- net at SW4.S2: now also D47.2 (A); no longer D47.1 (K)
- net at MX55.2 (ROW): now also D55.2 (A); no longer D55.1 (K)
- net at MX32.2 (ROW): now also D32.2 (A); no longer D32.1 (K)
- net at MX75.2 (ROW): now also D75.2 (A); no longer D75.1 (K)
- net at MX3.2 (ROW): now also D3.2 (A); no longer D3.1 (K)
- net at MX31.2 (ROW): now also D31.2 (A); no longer D31.1 (K)
- net at MX43.2 (ROW): now also D43.2 (A); no longer D43.1 (K)
- net at MX59.2 (ROW): now also D59.2 (A); no longer D59.1 (K)
- net at MX14.2 (ROW): now also D14.2 (A); no longer D14.1 (K)
- net at MX2.2 (ROW): now also D2.2 (A); no longer D2.1 (K)
- net at MX17.2 (ROW): now also D17.2 (A); no longer D17.1 (K)
- net at MX61.2 (ROW): now also D61.2 (A); no longer D61.1 (K)
- net at MX28.2 (ROW): now also D28.2 (A); no longer D28.1 (K)
- net at MX39.2 (ROW): now also D39.2 (A); no longer D39.1 (K)
- net at MX8.2 (ROW): now also D8.2 (A); no longer D8.1 (K)
- net at MX57.2 (ROW): now also D57.2 (A); no longer D57.1 (K)
- net at MX73.2 (ROW): now also D73.2 (A); no longer D73.1 (K)
- net at MX56.2 (ROW): now also D56.2 (A); no longer D56.1 (K)
- net at MX33.2 (ROW): now also D33.2 (A); no longer D33.1 (K)
- net at MX41.2 (ROW): now also D41.2 (A); no longer D41.1 (K)
- net at MX42.2 (ROW): now also D42.2 (A); no longer D42.1 (K)
- net at MX65.2 (ROW): now also D65.2 (A); no longer D65.1 (K)
- net at MX6.2 (ROW): now also D6.2 (A); no longer D6.1 (K)
- net at MX72.2 (ROW): now also D72.2 (A); no longer D72.1 (K)
- net at MX9.2 (ROW): now also D9.2 (A); no longer D9.1 (K)
- net at MX15.2 (ROW): now also D15.2 (A); no longer D15.1 (K)
- net at MX67.2 (ROW): now also D67.2 (A); no longer D67.1 (K)
- net at MX19.2 (ROW): now also D19.2 (A); no longer D19.1 (K)
- new net: D40.2 (A), MX40.2 (ROW)
- new net: D68.2 (A), MX68.2 (ROW)
- new net: D21.2 (A), MX21.2 (ROW)
- new net: D12.2 (A), MX12.2 (ROW)
- new net: D51.2 (A), MX51.2 (ROW)
- new net: D25.2 (A), MX25.2 (ROW)
- new net: D46.2 (A), MX46.2 (ROW)
- new net: D60.2 (A), MX60.2 (ROW)
- new net: D5.2 (A), MX5.2 (ROW)
- new net: D63.2 (A), MX63.2 (ROW)
Other:
- moved on the sheet: D1, D10, D11, D12, D13, D14, D15, D16, D17, D18, D19, D2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
